File: 170V升压电路/原理图.brd (EAGLE design)
At the start: 100 x 80 mm, 20 parts, among them IC1 MC34063AP

Commit message: 修改美化一下
Parts:
- moved VT14 17.0 mm to (40.6, 11.4), turned to 270 degrees
- moved C5 14.4 mm to (52.1, 33.0), turned to 90 degrees
- moved GND10 13.7 mm to (6.35, 38.1)
- moved VOUT170 13.7 mm to (8.89, 38.1)
- moved VD3 12.7 mm to (48.3, 25.4), turned to 270 degrees
- moved R21 11.4 mm to (27.9, 12.7)
- moved R23 11.4 mm to (22.9, 35.6)
- moved R22 9.16 mm to (33.0, 35.6)
- moved C8 7.62 mm to (12.7, 33.0)
- moved C7 7.62 mm to (41.9, 35.6)
- moved VT15 7.18 mm to (30.5, 20.3)
- moved R24 7.18 mm to (34.3, 27.9)
- moved C9 5.68 mm to (7.62, 26.7)
- moved L1 5.68 mm to (20.3, 8.89)
- moved VT13 5.68 mm to (40.6, 20.3)
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Routing:
- net N$4: track 74.7 -> 35.5 mm
- net +12V: track 83.7 -> 109.1 mm
- net +UB: track 50.0 -> 73.0 mm
- net N$2: track 14.3 -> 25.8 mm
- net N$8: track 17.0 -> 7.93 mm
- net GND: track 150.7 -> 145.8 mm
- net N$3: track 18.5 -> 23.3 mm
- net N$5: track 33.9 -> 30.0 mm
- net N$7: track 13.3 -> 16.8 mm
- net N$6: track 28.1 -> 31.4 mm
- net N$1: track 7.93 -> 8.98 mm

Commit message: 优化
Parts:
- renumbered VOUT170 to 170+
Changed lines of the file:
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@@
 <layer number="17" name="Pads" color="2" fill="1" visible="yes" active="yes"/>
 <layer number="18" name="Vias" color="2" fill="1" visible="yes" active="yes"/>
-<layer number="19" name="Unrouted" color="6" fill="1" visible="no" active="yes"/>
-<layer number="20" name="Dimension" color="15" fill="1" visible="no" active="yes"/>
-<layer number="21" name="tPlace" color="7" fill="1" visible="no" active="yes"/>
-<layer number="22" name="bPlace" color="7" fill="1" visible="no" active="yes"/>
-<layer number="23" name="tOrigins" color="15" fill="1" visible="no" active="yes"/>
-<layer number="24" name="bOrigins" color="15" fill="1" visible="no" active="yes"/>
-<layer number="25" name="tNames" color="7" fill="1" visible="no" active="yes"/>
-<layer number="26" name="bNames" color="7" fill="1" visible="no" active="yes"/>
-<layer number="27" name="tValues" color="7" fill="1" visible="no" active="yes"/>
-<layer number="28" name="bValues" color="7" fill="1" visible="no" active="yes"/>
-<layer number="29" name="tStop" color="7" fill="3" visible="no" active="yes"/>
-<layer number="30" name="bStop" color="7" fill="6" visible="no" active="yes"/>
-<layer number="31" name="tCream" color="7" fill="4" visible="no" active="yes"/>
-<layer number="32" name="bCream" color="7" fill="5" visible="no" active="yes"/>
-<layer number="33" name="tFinish" color="6" fill="3" visible="no" active="yes"/>
-<layer number="34" name="bFinish" color="6" fill="6" visible="no" active="yes"/>
-<layer number="35" name="tGlue" color="7" fill="4" visible="no" active="yes"/>
-<layer number="36" name="bGlue" color="7" fill="5" visible="no" active="yes"/>
-<layer number="37" name="tTest" color="7" fill="1" visible="no" active="yes"/>
-<layer number="38" name="bTest" color="7" fill="1" visible="no" active="yes"/>
-<layer number="39" name="tKeepout" color="4" fill="11" visible="no" active="yes"/>
-<layer number="40" name="bKeepout" color="1" fill="11" visible="no" active="yes"/>
-<layer number="41" name="tRestrict" color="4" fill="10" visible="no" active="yes"/>
-<layer number="42" name="bRestrict" color="1" fill="10" visible="no" active="yes"/>
-<layer number="43" name="vRestrict" color="2" fill="10" visible="no" active="yes"/>
-<layer number="44" name="Drills" color="7" fill="1" visible="no" active="yes"/>
-<layer number="45" name="Holes" color="7" fill="1" visible="no" active="yes"/>
-<layer number="46" name="Milling" color="3" fill="1" visible="no" active="yes"/>
-<layer number="47" name="Measures" color="7" fill="1" visible="no" active="yes"/>
-<layer number="48" name="Document" color="7" fill="1" visible="no" active="yes"/>
-<layer number="49" name="Reference" color="7" fill="1" visible="no" active="yes"/>
+<layer number="19" name="Unrouted" color="6" fill="1" visible="yes" active="yes"/>
+<layer number="20" name="Dimension" color="15" fill="1" visible="yes" active="yes"/>
+<layer number="21" name="tPlace" color="7" fill="1" visible="yes" active="yes"/>
+<layer number="22" name="bPlace" color="7" fill="1" visible="yes" active="yes"/>
+<layer number="23" name="tOrigins" color="15" fill="1" visible="yes" active="yes"/>
+<layer number="24" name="bOrigins" color="15" fill="1" visible="yes" active="yes"/>
+<layer number="25" name="tNames" color="7" fill="1" visible="yes" active="yes"/>
+<layer number="26" name="bNames" color="7" fill="1" visible="yes" active="yes"/>
+<layer number="27" name="tValues" color="7" fill="1" visible="yes" active="yes"/>
+<layer number="28" name="bValues" color="7" fill="1" visible="yes" active="yes"/>
+<layer number="29" name="tStop" color="7" fill="3" visible="yes" active="yes"/>
+<layer number="30" name="bStop" color="7" fill="6" visible="yes" active="yes"/>
+<layer number="31" name="tCream" color="7" fill="4" visible="yes" active="yes"/>
+<layer number="32" name="bCream" color="7" fill="5" visible="yes" active="yes"/>
+<layer number="33" name="tFinish" color="6" fill="3" visible="yes" active="yes"/>
+<layer number="34" name="bFinish" color="6" fill="6" visible="yes" active="yes"/>
+<layer number="35" name="tGlue" color="7" fill="4" visible="yes" active="yes"/>
+<layer number="36" name="bGlue" color="7" fill="5" visible="yes" active="yes"/>
+<layer number="37" name="tTest" color="7" fill="1" visible="yes" active="yes"/>
+<layer number="38" name="bTest" color="7" fill="1" visible="yes" active="yes"/>
+<layer number="39" name="tKeepout" color="4" fill="11" visible="yes" active="yes"/>
+<layer number="40" name="bKeepout" color="1" fill="11" visible="yes" active="yes"/>
+<layer number="41" name="tRestrict" color="4" fill="10" visible="yes" active="yes"/>
+<layer number="42" name="bRestrict" color="1" fill="10" visible="yes" active="yes"/>
+<layer number="43" name="vRestrict" color="2" fill="10" visible="yes" active="yes"/>
+<layer number="44" name="Drills" color="7" fill="1" visible="yes" active="yes"/>
+<layer number="45" name="Holes" color="7" fill="1" visible="yes" active="yes"/>
+<layer number="46" name="Milling" color="3" fill="1" visible="yes" active="yes"/>
+<layer number="47" name="Measures" color="7" fill="1" visible="yes" active="yes"/>
+<layer number="48" name="Document" color="7" fill="1" visible="yes" active="yes"/>
+<layer number="49" name="Reference" color="7" fill="1" visible="yes" active="yes"/>
 <layer number="50" name="dxf" color="7" fill="1" visible="no" active="no"/>
-<layer number="51" name="tDocu" color="7" fill="1" visible="no" active="yes"/>
-<layer number="52" name="bDocu" color="7" fill="1" visible="no" active="yes"/>
+<layer number="51" name="tDocu" color="7" fill="1" visible="yes" active="yes"/>
+<layer number="52" name="bDocu" color="7" fill="1" visible="yes" active="yes"/>
 <layer number="91" name="Nets" color="2" fill="1" visible="no" active="no"/>
 <layer number="92" name="Busses" color="1" fill="1" visible="no" active="no"/>
@@
 <layer number="97" name="Info" color="7" fill="1" visible="no" active="no"/>
 <layer number="98" name="Guide" color="6" fill="1" visible="no" active="no"/>
-<layer number="200" name="200bmp" color="7" fill="1" visible="no" active="yes"/>
-<layer number="231" name="Eagle3D_PG1" color="7" fill="1" visible="no" active="yes"/>
-<layer number="232" name="Eagle3D_PG2" color="7" fill="1" visible="no" active="yes"/>
-<layer number="233" name="Eagle3D_PG3" color="7" fill="1" visible="no" active="yes"/>
-<layer number="250" name="Descript" color="7" fill="1" visible="no" active="yes"/>
-<layer number="251" name="SMDround" color="7" fill="1" visible="no" active="yes"/>
+<layer number="200" name="200bmp" color="7" fill="1" visible="yes" active="yes"/>
+<layer number="231" name="Eagle3D_PG1" color="7" fill="1" visible="yes" active="yes"/>
+<layer number="232" name="Eagle3D_PG2" color="7" fill="1" visible="yes" active="yes"/>
+<layer number="233" name="Eagle3D_PG3" color="7" fill="1" visible="yes" active="yes"/>
+<layer number="250" name="Descript" color="7" fill="1" visible="yes" active="yes"/>
+<layer number="251" name="SMDround" color="7" fill="1" visible="yes" active="yes"/>
 </layers>
 <board>
@@
 <attribute name="VALUE" x="7.62" y="5.68" size="0.0254" layer="27"/>
 </element>
-<element name="VOUT170" library="wirepad" package="2,54/0,8" value="" x="8.89" y="38.1" smashed="yes">
+<element name="170+" library="wirepad" package="2,54/0,8" value="" x="8.89" y="38.1" smashed="yes">
 <attribute name="NAME" x="7.62" y="39.624" size="1.27" layer="25" ratio="10"/>
 <attribute name="VALUE" x="8.89" y="38.7" size="0.0254" layer="27"/>
@@
 <contactref element="VD3" pad="C"/>
 <contactref element="C5" pad="1"/>
-<contactref element="VOUT170" pad="1"/>
+<contactref element="170+" pad="1"/>
 <wire x1="40.64" y1="30.48" x2="35.56" y2="35.56" width="0.254" layer="1"/>
 <wire x1="48.26" y1="30.48" x2="40.64" y2="30.48" width="0.254" layer="1"/>

Commit message: 哈哈  有点好看了。
Parts:
- moved GND 1.27 mm to (6.35, 5.08)
- moved VCC 1.27 mm to (8.89, 5.08)
Routing:
- net +12V: track 109.1 -> 86.7 mm
- net GND: track 145.8 -> 156.7 mm
Changed lines of the file:
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@@
 <element name="R21" library="rcl" package="0204/5" value="18" x="27.94" y="12.7" rot="R270"/>
 <element name="C5" library="rcl" package="C025-030X050" value="4.7u 250V" x="52.07" y="33.02" rot="R90"/>
-<element name="VCC" library="wirepad" package="2,54/0,8" value="" x="10.16" y="5.08"/>
-<element name="GND" library="wirepad" package="2,54/0,8" value="" x="7.62" y="5.08" smashed="yes">
-<attribute name="NAME" x="6.35" y="6.604" size="1.27" layer="25" ratio="10"/>
-<attribute name="VALUE" x="7.62" y="5.68" size="0.0254" layer="27"/>
+<element name="VCC" library="wirepad" package="2,54/0,8" value="" x="8.89" y="5.08"/>
+<element name="GND" library="wirepad" package="2,54/0,8" value="" x="6.35" y="5.08" smashed="yes">
+<attribute name="NAME" x="5.08" y="6.604" size="1.27" layer="25" ratio="10"/>
+<attribute name="VALUE" x="6.35" y="5.68" size="0.0254" layer="27"/>
 </element>
 <element name="170+" library="wirepad" package="2,54/0,8" value="" x="8.89" y="38.1" smashed="yes">
@@
 <wire x1="21.59" y1="27.94" x2="24.13" y2="27.94" width="0.254" layer="1"/>
 <wire x1="17.78" y1="26.67" x2="19.05" y2="27.94" width="0.254" layer="1"/>
-<wire x1="7.62" y1="26.67" x2="8.89" y2="26.67" width="0.254" layer="1"/>
-<wire x1="8.89" y1="26.67" x2="17.78" y2="26.67" width="0.254" layer="1"/>
+<wire x1="7.62" y1="26.67" x2="17.78" y2="26.67" width="0.254" layer="1"/>
 <wire x1="7.62" y1="27.94" x2="7.62" y2="26.67" width="0.254" layer="1"/>
 <wire x1="26.67" y1="8.89" x2="34.29" y2="8.89" width="0.254" layer="1"/>
@@
 <wire x1="21.59" y1="27.94" x2="21.59" y2="24.13" width="0.254" layer="1"/>
 <wire x1="21.59" y1="24.13" x2="21.59" y2="21.59" width="0.254" layer="1"/>
-<wire x1="8.89" y1="6.35" x2="7.62" y2="5.08" width="0.254" layer="1"/>
-<wire x1="8.89" y1="26.67" x2="8.89" y2="6.35" width="0.254" layer="1"/>
 <wire x1="11.43" y1="33.02" x2="6.35" y2="38.1" width="0.254" layer="1"/>
 <wire x1="21.59" y1="24.13" x2="31.75" y2="24.13" width="0.254" layer="1"/>
@@
 <wire x1="34.29" y1="30.48" x2="34.29" y2="36.83" width="0.254" layer="1"/>
 <wire x1="31.75" y1="27.94" x2="34.29" y2="30.48" width="0.254" layer="1"/>
+<wire x1="6.35" y1="38.1" x2="6.35" y2="5.08" width="0.254" layer="1"/>
 </signal>
 <signal name="+12V">
@@
 <contactref element="VT13" pad="1"/>
 <contactref element="IC1" pad="6"/>
-<wire x1="5.08" y1="22.86" x2="7.62" y2="25.4" width="0.254" layer="1"/>
-<wire x1="5.08" y1="5.08" x2="5.08" y2="22.86" width="0.254" layer="1"/>
-<wire x1="7.62" y1="2.54" x2="5.08" y2="5.08" width="0.254" layer="1"/>
-<wire x1="10.16" y1="2.54" x2="7.62" y2="2.54" width="0.254" layer="1"/>
-<wire x1="10.16" y1="5.08" x2="10.16" y2="2.54" width="0.254" layer="1"/>
-<wire x1="10.16" y1="15.24" x2="12.7" y2="17.78" width="0.254" layer="1"/>
-<wire x1="10.16" y1="5.08" x2="10.16" y2="6.35" width="0.254" layer="1"/>
-<wire x1="10.16" y1="6.35" x2="10.16" y2="15.24" width="0.254" layer="1"/>
 <wire x1="46.99" y1="20.32" x2="41.91" y2="20.32" width="0.254" layer="1"/>
 <wire x1="46.99" y1="21.59" x2="46.99" y2="20.32" width="0.254" layer="1"/>
@@
 <wire x1="49.53" y1="19.05" x2="49.53" y2="21.59" width="0.254" layer="1"/>
 <wire x1="36.83" y1="6.35" x2="49.53" y2="19.05" width="0.254" layer="1"/>
+<wire x1="12.7" y1="21.59" x2="16.51" y2="25.4" width="0.254" layer="1"/>
+<wire x1="12.7" y1="17.78" x2="12.7" y2="20.32" width="0.254" layer="1"/>
+<wire x1="12.7" y1="20.32" x2="12.7" y2="21.59" width="0.254" layer="1"/>
+<wire x1="12.7" y1="20.32" x2="7.62" y2="25.4" width="0.254" layer="1"/>
+<wire x1="10.16" y1="15.24" x2="12.7" y2="17.78" width="0.254" layer="1"/>
+<wire x1="8.89" y1="5.08" x2="10.16" y2="6.35" width="0.254" layer="1"/>
 <wire x1="10.16" y1="6.35" x2="36.83" y2="6.35" width="0.254" layer="1"/>
-<wire x1="12.7" y1="21.59" x2="16.51" y2="25.4" width="0.254" layer="1"/>
-<wire x1="12.7" y1="17.78" x2="12.7" y2="21.59" width="0.254" layer="1"/>
+<wire x1="10.16" y1="6.35" x2="10.16" y2="15.24" width="0.254" layer="1"/>
 </signal>
 <signal name="N$2">

Commit message: 持续优化
Parts:
- moved 170+ 1.27 mm to (10.2, 38.1)
- moved VCC 1.27 mm to (10.2, 5.08)
Routing:
- net GND: track 156.7 -> 152.4 mm
- net +UB: track 73.0 -> 71.7 mm
- net +12V: track 86.7 -> 86.2 mm
Changed lines of the file:
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@@
 <element name="R21" library="rcl" package="0204/5" value="18" x="27.94" y="12.7" rot="R270"/>
 <element name="C5" library="rcl" package="C025-030X050" value="4.7u 250V" x="52.07" y="33.02" rot="R90"/>
-<element name="VCC" library="wirepad" package="2,54/0,8" value="" x="8.89" y="5.08"/>
+<element name="VCC" library="wirepad" package="2,54/0,8" value="" x="10.16" y="5.08"/>
 <element name="GND" library="wirepad" package="2,54/0,8" value="" x="6.35" y="5.08" smashed="yes">
 <attribute name="NAME" x="5.08" y="6.604" size="1.27" layer="25" ratio="10"/>
 <attribute name="VALUE" x="6.35" y="5.68" size="0.0254" layer="27"/>
 </element>
-<element name="170+" library="wirepad" package="2,54/0,8" value="" x="8.89" y="38.1" smashed="yes">
-<attribute name="NAME" x="7.62" y="39.624" size="1.27" layer="25" ratio="10"/>
-<attribute name="VALUE" x="8.89" y="38.7" size="0.0254" layer="27"/>
+<element name="170+" library="wirepad" package="2,54/0,8" value="" x="10.16" y="38.1" smashed="yes">
+<attribute name="NAME" x="8.89" y="39.624" size="1.27" layer="25" ratio="10"/>
+<attribute name="VALUE" x="10.16" y="38.7" size="0.0254" layer="27"/>
 </element>
 <element name="GND10" library="wirepad" package="2,54/0,8" value="" x="6.35" y="38.1" smashed="yes">
@@
 <wire x1="52.07" y1="35.56" x2="43.18" y2="35.56" width="0.254" layer="1"/>
 <wire x1="52.07" y1="34.29" x2="52.07" y2="35.56" width="0.254" layer="1"/>
-<wire x1="31.75" y1="27.94" x2="31.75" y2="24.13" width="0.254" layer="1"/>
-<wire x1="31.75" y1="24.13" x2="31.75" y2="20.32" width="0.254" layer="1"/>
-<wire x1="11.43" y1="31.75" x2="7.62" y2="27.94" width="0.254" layer="1"/>
-<wire x1="11.43" y1="33.02" x2="11.43" y2="31.75" width="0.254" layer="1"/>
-<wire x1="11.43" y1="35.56" x2="20.32" y2="35.56" width="0.254" layer="1"/>
-<wire x1="11.43" y1="33.02" x2="11.43" y2="35.56" width="0.254" layer="1"/>
-<wire x1="19.05" y1="27.94" x2="21.59" y2="27.94" width="0.254" layer="1"/>
-<wire x1="21.59" y1="27.94" x2="24.13" y2="27.94" width="0.254" layer="1"/>
-<wire x1="17.78" y1="26.67" x2="19.05" y2="27.94" width="0.254" layer="1"/>
-<wire x1="7.62" y1="26.67" x2="17.78" y2="26.67" width="0.254" layer="1"/>
-<wire x1="7.62" y1="27.94" x2="7.62" y2="26.67" width="0.254" layer="1"/>
-<wire x1="26.67" y1="8.89" x2="34.29" y2="8.89" width="0.254" layer="1"/>
-<wire x1="26.67" y1="20.32" x2="26.67" y2="8.89" width="0.254" layer="1"/>
-<wire x1="25.4" y1="21.59" x2="26.67" y2="20.32" width="0.254" layer="1"/>
-<wire x1="21.59" y1="21.59" x2="25.4" y2="21.59" width="0.254" layer="1"/>
-<wire x1="21.59" y1="27.94" x2="21.59" y2="24.13" width="0.254" layer="1"/>
-<wire x1="21.59" y1="24.13" x2="21.59" y2="21.59" width="0.254" layer="1"/>
-<wire x1="11.43" y1="33.02" x2="6.35" y2="38.1" width="0.254" layer="1"/>
-<wire x1="21.59" y1="24.13" x2="31.75" y2="24.13" width="0.254" layer="1"/>
 <wire x1="41.91" y1="34.29" x2="43.18" y2="35.56" width="0.254" layer="1"/>
 <wire x1="38.1" y1="34.29" x2="41.91" y2="34.29" width="0.254" layer="1"/>
@@
 <wire x1="34.29" y1="30.48" x2="34.29" y2="36.83" width="0.254" layer="1"/>
 <wire x1="31.75" y1="27.94" x2="34.29" y2="30.48" width="0.254" layer="1"/>
-<wire x1="6.35" y1="38.1" x2="6.35" y2="5.08" width="0.254" layer="1"/>
+<wire x1="6.35" y1="38.1" x2="6.35" y2="26.67" width="0.254" layer="1"/>
+<wire x1="6.35" y1="26.67" x2="6.35" y2="5.08" width="0.254" layer="1"/>
+<wire x1="31.75" y1="27.94" x2="31.75" y2="20.32" width="0.254" layer="1"/>
+<wire x1="11.43" y1="31.75" x2="7.62" y2="27.94" width="0.254" layer="1"/>
+<wire x1="11.43" y1="33.02" x2="11.43" y2="31.75" width="0.254" layer="1"/>
+<wire x1="19.05" y1="27.94" x2="21.59" y2="27.94" width="0.254" layer="1"/>
+<wire x1="21.59" y1="27.94" x2="24.13" y2="27.94" width="0.254" layer="1"/>
+<wire x1="17.78" y1="26.67" x2="19.05" y2="27.94" width="0.254" layer="1"/>
+<wire x1="7.62" y1="26.67" x2="17.78" y2="26.67" width="0.254" layer="1"/>
+<wire x1="7.62" y1="27.94" x2="7.62" y2="26.67" width="0.254" layer="1"/>
+<wire x1="11.43" y1="35.56" x2="20.32" y2="35.56" width="0.254" layer="1"/>
+<wire x1="11.43" y1="33.02" x2="11.43" y2="35.56" width="0.254" layer="1"/>
+<wire x1="26.67" y1="8.89" x2="34.29" y2="8.89" width="0.254" layer="1"/>
+<wire x1="26.67" y1="20.32" x2="26.67" y2="8.89" width="0.254" layer="1"/>
+<wire x1="25.4" y1="21.59" x2="26.67" y2="20.32" width="0.254" layer="1"/>
+<wire x1="21.59" y1="21.59" x2="25.4" y2="21.59" width="0.254" layer="1"/>
+<wire x1="21.59" y1="27.94" x2="21.59" y2="24.13" width="0.254" layer="1"/>
+<wire x1="21.59" y1="24.13" x2="21.59" y2="21.59" width="0.254" layer="1"/>
+<wire x1="27.94" y1="24.13" x2="31.75" y2="27.94" width="0.254" layer="1"/>
+<wire x1="21.59" y1="24.13" x2="27.94" y2="24.13" width="0.254" layer="1"/>
+<wire x1="7.62" y1="26.67" x2="6.35" y2="26.67" width="0.254" layer="1"/>
 </signal>
 <signal name="+12V">
@@
 <contactref element="VT13" pad="1"/>
 <contactref element="IC1" pad="6"/>
+<wire x1="12.7" y1="21.59" x2="16.51" y2="25.4" width="0.254" layer="1"/>
+<wire x1="12.7" y1="17.78" x2="12.7" y2="20.32" width="0.254" layer="1"/>
+<wire x1="12.7" y1="20.32" x2="12.7" y2="21.59" width="0.254" layer="1"/>
+<wire x1="12.7" y1="20.32" x2="7.62" y2="25.4" width="0.254" layer="1"/>
 <wire x1="46.99" y1="20.32" x2="41.91" y2="20.32" width="0.254" layer="1"/>
 <wire x1="46.99" y1="21.59" x2="46.99" y2="20.32" width="0.254" layer="1"/>
 <wire x1="49.53" y1="21.59" x2="46.99" y2="21.59" width="0.254" layer="1"/>
 <wire x1="49.53" y1="19.05" x2="49.53" y2="21.59" width="0.254" layer="1"/>
-<wire x1="36.83" y1="6.35" x2="49.53" y2="19.05" width="0.254" layer="1"/>
-<wire x1="12.7" y1="21.59" x2="16.51" y2="25.4" width="0.254" layer="1"/>
-<wire x1="12.7" y1="17.78" x2="12.7" y2="20.32" width="0.254" layer="1"/>
-<wire x1="12.7" y1="20.32" x2="12.7" y2="21.59" width="0.254" layer="1"/>
-<wire x1="12.7" y1="20.32" x2="7.62" y2="25.4" width="0.254" layer="1"/>
-<wire x1="10.16" y1="15.24" x2="12.7" y2="17.78" width="0.254" layer="1"/>
-<wire x1="8.89" y1="5.08" x2="10.16" y2="6.35" width="0.254" layer="1"/>
-<wire x1="10.16" y1="6.35" x2="36.83" y2="6.35" width="0.254" layer="1"/>
-<wire x1="10.16" y1="6.35" x2="10.16" y2="15.24" width="0.254" layer="1"/>
+<wire x1="35.56" y1="5.08" x2="49.53" y2="19.05" width="0.254" layer="1"/>
+<wire x1="10.16" y1="5.08" x2="11.43" y2="5.08" width="0.254" layer="1"/>
+<wire x1="11.43" y1="5.08" x2="35.56" y2="5.08" width="0.254" layer="1"/>
+<wire x1="11.43" y1="16.51" x2="12.7" y2="17.78" width="0.254" layer="1"/>
+<wire x1="11.43" y1="5.08" x2="11.43" y2="16.51" width="0.254" layer="1"/>
 </signal>
 <signal name="N$2">
@@
 <wire x1="48.26" y1="31.75" x2="52.07" y2="31.75" width="0.254" layer="1"/>
 <wire x1="48.26" y1="30.48" x2="48.26" y2="31.75" width="0.254" layer="1"/>
-<wire x1="33.02" y1="38.1" x2="8.89" y2="38.1" width="0.254" layer="1"/>
+<wire x1="33.02" y1="38.1" x2="10.16" y2="38.1" width="0.254" layer="1"/>
 <wire x1="34.29" y1="39.37" x2="33.02" y2="38.1" width="0.254" layer="1"/>
 <wire x1="53.34" y1="39.37" x2="34.29" y2="39.37" width="0.254" layer="1"/>
