File: 170V升压电路/升压.brd (EAGLE design)
At the start: 100 x 80 mm, 20 parts, among them IC1 MC34063AP

Commit message: 修改电容元器件的尺寸
Parts:
- C5, C7, C8, C9: device rcl:C025-030X050 -> rcl:C050-025X075
- L1: device rcl:0204/5 -> rcl:0207/10
- moved L1 2.54 mm to (20.3, 6.35)
Routing:
- net N$2: track 25.8 -> 22.0 mm
- net GND: track 152.4 -> 155.6 mm
- net N$5: track 30.0 -> 32.4 mm
- net N$4: track 35.5 -> 33.7 mm
- net +12V: track 86.2 -> 87.5 mm
- net N$3: track 23.3 -> 22.4 mm
